Commit message: Gazebo: rviz-only material tags now apply to models in Gazebo

File: pbr_gazebo/urdf/box.gazebo.xacro (robot description, xacro)
@@ -8,5 +8,5 @@
           <box size="${width} ${length} ${height}"/>
         </geometry>
-        <material name="orange"> <!-- rviz will use this color -->
+        <material name="orange">
           <color rgba="${255/255} ${108/255} ${10/255} 1.0"/>
         </material>
@@ -26,7 +26,4 @@
       </inertial>
     </link>
-    <gazebo reference="${name}_box">
-      <material>Gazebo/${color}</material> <!-- gazebo will use this color -->
-    </gazebo>
   </xacro:macro>
   <!-- example on how to call this macro -->

File: pbr_gazebo/urdf/rgb_camera.gazebo.xacro (robot description, xacro)
@@ -7,4 +7,7 @@
           <cylinder length="0.01" radius="0.03"/>
         </geometry>
+        <material name="light_green">
+          <color rgba="0 1 0 0.3"/>
+        </material>
       </visual>
       <collision>
@@ -21,7 +24,4 @@
       </inertial>
     </link>
-    <gazebo reference="${camera_name}_link">
-      <material>Gazebo/GreenTransparent</material>
-    </gazebo>
     <link name="${camera_name}_box_link">
       <visual>
@@ -29,4 +29,7 @@
           <box size="0.1 0.1 0.03"/>
         </geometry>
+        <material name="grey">
+          <color rgba="0.5 0.5 0.5 1"/>
+        </material>
       </visual>
       <collision>
@@ -43,7 +46,4 @@
       </inertial>
     </link>
-    <gazebo reference="${camera_name}_box_link">
-      <material>Gazebo/Gray</material>
-    </gazebo>
     <joint name="${camera_name}_box_link_to_${camera_name}_link" type="fixed">
       <parent link="${camera_name}_box_link"/>
